File: ESPeranza8266/ESPeranza8266.sch (KiCad schematic (older format))
At the start: 31 parts, among them J1 GS1, J11 Conn_01x10_Male, J12 Conn_01x04, J13 Conn_01x04, J14 Conn_01x02, J15 Conn_01x03, J16 Conn_01x02, J17 Conn_01x02, J18 Conn_01x01_Male, J3 GS3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

Commit message: added RXD (D9) to jumper J1 changed fontsizes and placements of component references
Parts:
- J1: symbol Conn_01x04 -> Conn_01x05
Connections:
- wire segments 110 -> 111
Changed lines of the file:
@@
 RST
 $Comp
-L Conn_01x04 J1
+L Conn_01x05 J1
 U 1 1 5A73348F
-P 10300 1600
-F 0 "J1" H 10300 1800 50  0000 C CNN
-F 1 "GS1" H 10300 1300 50  0000 C CNN
-F 2 "GS4-SQUARE" V 10374 1600 50  0001 C CNN
-F 3 "" H 10300 1600 50  0001 C CNN
-	1    10300 1600
+P 10300 1700
+F 0 "J1" H 10300 1900 50  0000 C CNN
+F 1 "GS1" H 10300 1400 50  0000 C CNN
+F 2 "GS4-SQUARE" V 10374 1700 50  0001 C CNN
+F 3 "" H 10300 1700 50  0001 C CNN
+	1    10300 1700
 	1    0    0    -1
 $EndComp
@@
 Text Label 8600 4650 2    60   ~ 0
 IO10
+Text GLabel 9850 1900 0    60   3State ~ 0
+RXD
+Wire Wire Line
+	10100 1900 9850 1900
 $EndSCHEMATC

Commit message: Added MCP73831 (battery charge management controller) and battery connector
Parts:
- removed J15: Conn_01x03, PERSONAL:GroundPad_01x03, symbol Conn_01x03
- removed J3: GS3, Connectors:GS3, symbol GS3
- removed J4: GS4, Connectors:GS3, symbol GS3
- added C7: 4.7uF, PERSONAL:SMD_1206_0805_Universal, symbol C
- added D3: Yellow, PERSONAL:SMD_1206_0805_Universal, symbol LED
- added D4: MBR120, Diodes_SMD:D_SOD-123, symbol D_Schottky
- added J10: USB_OTG, symbol USB_OTG
- added J19: LiPo, Connectors_JST:JST_EH_S02B-EH_02x2.50mm_Angled, symbol Conn_01x02
- added R10: 2.0k, PERSONAL:SMD_1206_0805_Universal, symbol R_Small
- added R9: 200, PERSONAL:SMD_1206_0805_Universal, symbol R_Small
- added U3: MCP73831, TO_SOT_Packages_SMD:SOT-23-5_HandSoldering, symbol MCP73831
- J14: symbol Conn_01x03 -> Conn_01x02
- J16: footprint PowerPad_01x03_R -> PowerPad_01x02_R; symbol Conn_01x03 -> Conn_01x02
Connections:
- net labels added: +BATT, PROG
- net labels removed: Vxx, Vyy
- wire segments 111 -> 119
- no-connect marks 2 -> 5
Other:
- moved on the sheet: C1, C2, C3, C4, C5, C6, D1, D2, J1, J11, J12, J13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
